File: Foras Promineo CLR PCB.kicad_pcb (KiCad board)
At the start: 2 copper layers, 39.8 x 39.8 mm, 27 parts, among them J1 Conn_01x10_Male

Commit message: assembly files
Parts:
- renumbered REF** to REFe
Changed lines of the file:
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@@
     (property "ki_description" "Light emitting diode")
     (property "ki_keywords" "LED diode")
-    (attr through_hole)
+    (attr smd)
     (fp_text reference "D2" (at -0.038816 -2.941427 10) (layer "F.SilkS")
         (effects (font (size 1 1) (thickness 0.15)))
     )
-    (fp_text value "LED" (at 0 0.27 -80) (layer "F.Fab")
+    (fp_text value "LED" (at 0 0.27 100) (layer "F.Fab")
         (effects (font (size 1 1) (thickness 0.15)))
     )
@@
     (property "ki_description" "Light emitting diode")
     (property "ki_keywords" "LED diode")
-    (attr through_hole)
+    (attr smd)
     (fp_text reference "D3" (at -3.397648 -0.405172 45) (layer "F.SilkS")
         (effects (font (size 1 1) (thickness 0.15)))
@@
     (property "ki_description" "Light emitting diode")
     (property "ki_keywords" "LED diode")
-    (attr through_hole)
+    (attr smd)
     (fp_text reference "D1" (at 3.749092 -0.489776 60.857) (layer "F.SilkS")
         (effects (font (size 1 1) (thickness 0.15)))
     )
-    (fp_text value "LED" (at 0 0.27 -29.143) (layer "F.Fab")
+    (fp_text value "LED" (at 0 0.27 150.857) (layer "F.Fab")
         (effects (font (size 1 1) (thickness 0.15)))
     )
@@
     (property "ki_description" "Light emitting diode")
     (property "ki_keywords" "LED diode")
-    (attr through_hole)
+    (attr smd)
     (fp_text reference "D5" (at 0.029532 -2.827078 80) (layer "F.SilkS")
         (effects (font (size 1 1) (thickness 0.15)))
@@
     (property "ki_description" "Light emitting diode")
     (property "ki_keywords" "LED diode")
-    (attr through_hole)
+    (attr smd)
     (fp_text reference "D6" (at -3.16357 -0.020536 30) (layer "F.SilkS")
         (effects (font (size 1 1) (thickness 0.15)))
@@
     (property "ki_description" "Light emitting diode")
     (property "ki_keywords" "LED diode")
-    (attr through_hole)
+    (attr smd)
     (fp_text reference "D4" (at 3.478965 0.140007 225) (layer "F.SilkS")
         (effects (font (size 1 1) (thickness 0.15)))
@@
     (descr "Circular Fiducial, 1mm bare copper, 3mm soldermask opening (recommended)")
     (tags "fiducial")
-    (attr smd)
+    (attr smd board_only exclude_from_pos_files exclude_from_bom)
     (fp_text reference "REF**" (at 0 -2.54 90) (layer "F.SilkS") hide
         (effects (font (size 1 1) (thickness 0.15)))
@@
     (descr "Circular Fiducial, 1mm bare copper, 3mm soldermask opening (recommended)")
     (tags "fiducial")
-    (attr smd)
+    (attr smd board_only exclude_from_pos_files exclude_from_bom)
     (fp_text reference "REF**" (at 0 -2.54 90) (layer "F.SilkS") hide
         (effects (font (size 1 1) (thickness 0.15)))
@@
     (descr "Circular Fiducial, 1mm bare copper, 3mm soldermask opening (recommended)")
     (tags "fiducial")
-    (attr smd)
+    (attr smd board_only exclude_from_pos_files exclude_from_bom)
     (fp_text reference "REF**" (at 0 -2.54 90) (layer "F.SilkS") hide
         (effects (font (size 1 1) (thickness 0.15)))
@@
     (property "ki_description" "Generic connector, single row, 01x10, script generated (kicad-library-utils/schlib/autogen/connector/)")
     (property "ki_keywords" "connector")
-    (attr through_hole)
+    (attr smd)
     (fp_text reference "J1" (at -4.9 -4.2 180) (layer "B.SilkS")
         (effects (font (size 1 1) (thickness 0.15)) (justify mirror))
@@
     (descr "Circular Fiducial, 1mm bare copper, 3mm soldermask opening (recommended)")
     (tags "fiducial")
-    (attr smd)
+    (attr smd board_only exclude_from_pos_files exclude_from_bom)
     (fp_text reference "REF**" (at 0 2.54) (layer "B.SilkS") hide
         (effects (font (size 1 1) (thickness 0.15)) (justify mirror))
@@
     (descr "Circular Fiducial, 1mm bare copper, 3mm soldermask opening (recommended)")
     (tags "fiducial")
-    (attr smd)
-    (fp_text reference "REF**" (at 0 2.54) (layer "B.SilkS") hide
+    (attr smd board_only exclude_from_pos_files exclude_from_bom)
+    (fp_text reference "REFe" (at 0 2.54) (layer "B.SilkS") hide
         (effects (font (size 1 1) (thickness 0.15)) (justify mirror))
     )
@@
     (descr "Circular Fiducial, 1mm bare copper, 3mm soldermask opening (recommended)")
     (tags "fiducial")
-    (attr smd)
+    (attr smd board_only exclude_from_pos_files exclude_from_bom)
     (fp_text reference "REF**" (at 0 2.54) (layer "B.SilkS") hide
         (effects (font (size 1 1) (thickness 0.15)) (justify mirror))
@@
     (height 10.749463)
     (orientation 0)
-    (gr_text "5.0700 mm" (at 97.465 103.049463) (layer "Eco1.User")
+    (gr_text "5.0700 mm" (at 105 104.2) (layer "Eco1.User")
       (effects (font (size 1 1) (thickness 0.15)))
     )
     (format (prefix "") (suffix "") (units 3) (units_format 1) (precision 4))
-    (style (thickness 0.1) (arrow_length 1.27) (text_position_mode 0) (extension_height 0.58642) (extension_offset 0.5) keep_text_aligned)
+    (style (thickness 0.1) (arrow_length 1.27) (text_position_mode 2) (extension_height 0.58642) (extension_offset 0.5) keep_text_aligned)
   )
   (dimension (type orthogonal) (layer "Eco1.User")
@@
     (height 7.4)
     (orientation 0)
-    (gr_text "5.2707 mm" (at 62.83535 106.25) (layer "Eco1.User")
+    (gr_text "5.2707 mm" (at 55 107.2) (layer "Eco1.User")
       (effects (font (size 1 1) (thickness 0.15)))
     )
     (format (prefix "") (suffix "") (units 3) (units_format 1) (precision 4))
-    (style (thickness 0.1) (arrow_length 1.27) (text_position_mode 0) (extension_height 0.58642) (extension_offset 0.5) keep_text_aligned)
+    (style (thickness 0.1) (arrow_length 1.27) (text_position_mode 2) (extension_height 0.58642) (extension_offset 0.5) keep_text_aligned)
   )
   (dimension (type orthogonal) (layer "Eco1.User")
@@
   (dimension (type orthogonal) (layer "Eco1.User")
     (pts (xy 62.2 98) (xy 60.2 100))
-    (height -5)
+    (height -10.4)
     (orientation 1)
-    (gr_text "2.0000 mm" (at 56.05 99 90) (layer "Eco1.User")
+    (gr_text "2.0000 mm" (at 50.4 98.8 90) (layer "Eco1.User")
       (effects (font (size 1 1) (thickness 0.15)))
     )
     (format (prefix "") (suffix "") (units 3) (units_format 1) (precision 4))
-    (style (thickness 0.1) (arrow_length 1.27) (text_position_mode 0) (extension_height 0.58642) (extension_offset 0.5) keep_text_aligned)
+    (style (thickness 0.1) (arrow_length 1.27) (text_position_mode 2) (extension_height 0.58642) (extension_offset 0.5) keep_text_aligned)
   )
   (dimension (type orthogonal) (layer "Eco1.User")
@@
     (height 11.4)
     (orientation 0)
-    (gr_text "39.8000 mm" (at 80.1 110.25) (layer "Eco1.User")
+    (gr_text "39.8000 mm" (at 74.2 110.2) (layer "Eco1.User")
       (effects (font (size 1 1) (thickness 0.15)))
     )
     (format (prefix "") (suffix "") (units 3) (units_format 1) (precision 4))
-    (style (thickness 0.1) (arrow_length 1.27) (text_position_mode 0) (extension_height 0.58642) (extension_offset 0.5) keep_text_aligned)
+    (style (thickness 0.1) (arrow_length 1.27) (text_position_mode 2) (extension_height 0.58642) (extension_offset 0.5) keep_text_aligned)
   )
   (dimension (type orthogonal) (layer "Eco1.User")
     (pts (xy 60.2 62.4) (xy 62.2 62))
-    (height -4.4)
+    (height -10.6)
     (orientation 0)
-    (gr_text "2.0000 mm" (at 61.2 56.85) (layer "Eco1.User")
+    (gr_text "2.0000 mm" (at 61.2 50.65) (layer "Eco1.User")
       (effects (font (size 1 1) (thickness 0.15)))
     )
@@
   )
   (dimension (type orthogonal) (layer "Eco1.User")
-    (pts (xy 60 60) (xy 96.2 62))
+    (pts (xy 60.2 60.2) (xy 96.2 63))
     (height -2.6)
     (orientation 0)
-    (gr_text "36.2000 mm" (at 78.1 56.25) (layer "Eco1.User")
+    (gr_text "36.0000 mm" (at 78.2 56.45) (layer "Eco1.User")
       (effects (font (size 1 1) (thickness 0.15)))
     )
@@
     (height 8.8)
     (orientation 0)
-    (gr_text "34.7300 mm" (at 77.565 107.65) (layer "Eco1.User")
+    (gr_text "34.7300 mm" (at 74.4 107.65) (layer "Eco1.User")
       (effects (font (size 1 1) (thickness 0.15)))
     )
     (format (prefix "") (suffix "") (units 3) (units_format 1) (precision 4))
-    (style (thickness 0.1) (arrow_length 1.27) (text_position_mode 0) (extension_height 0.58642) (extension_offset 0.5) keep_text_aligned)
+    (style (thickness 0.1) (arrow_length 1.27) (text_position_mode 2) (extension_height 0.58642) (extension_offset 0.5) keep_text_aligned)
   )
   (dimension (type orthogonal) (layer "Eco1.User")
@@
     (height 4.4)
     (orientation 0)
-    (gr_text "2.0000 mm" (at 61.2 103.45) (layer "Eco1.User")
+    (gr_text "2.0000 mm" (at 55.4 104.6) (layer "Eco1.User")
       (effects (font (size 1 1) (thickness 0.15)))
     )
     (format (prefix "") (suffix "") (units 3) (units_format 1) (precision 4))
-    (style (thickness 0.1) (arrow_length 1.27) (text_position_mode 0) (extension_height 0.58642) (extension_offset 0.5) keep_text_aligned)
+    (style (thickness 0.1) (arrow_length 1.27) (text_position_mode 2) (extension_height 0.58642) (extension_offset 0.5) keep_text_aligned)
   )
   (segment (start 73.5 65.5375) (end 73.5 64.6375) (width 0.6) (layer "F.Cu") (net 1))
