File: Foras Promineo CLR PCB.kicad_sch (KiCad schematic)
At the start: 19 parts, among them J1 Conn_01x10_Male

Commit message: FM DONE!
Parts:
- D3: footprint Foras_Promineo:1212_LED_Pol_End -> Foras_Promineo_Github_Local:1212_LED_Pol
Other:
- note removed: "T1M-05-GF-DV CHANGE FOOTPRINT"
- company: (none) -> FRC ROBOTICS TEAM
- moved on the sheet: C1, C2, C5, C6, D1, D2, D3, D4, D5, D6, H1, H2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

Commit message: moved mounting holes and added fiducials
Parts:
- H1, H2: footprint MountingHole:MountingHole_3.5mm_Pad_Via -> MountingHole:MountingHole_2.7mm_M2.5_DIN965_Pad

Commit message: assembly files
Parts:
- H1, H2: now left out of the parts list
- J1: Manufacturer Hirose Electric Co Ltd -> Samtec; Manufacturer Part Number DF13-10P-1.25DSA -> T1M-05-GF-DV-K; Supplier Part Number H2198-ND -> SAM15304DKR-ND
Changed lines of the file:
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@@
   )
   (symbol (lib_id "Mechanical:MountingHole_Pad") (at 210.82 146.05 0) (unit 1)
-    (in_bom yes) (on_board yes) (dnp no)
+    (in_bom no) (on_board yes) (dnp no)
     (property "Reference" "H1" (at 213.36 144.8054 0)
       (effects (font (size 1.27 1.27)) (justify left))
@@
   )
   (symbol (lib_id "Mechanical:MountingHole_Pad") (at 234.95 146.05 0) (unit 1)
-    (in_bom yes) (on_board yes) (dnp no)
+    (in_bom no) (on_board yes) (dnp no)
     (property "Reference" "H2" (at 237.49 144.8054 0)
       (effects (font (size 1.27 1.27)) (justify left))
@@
       (effects (font (size 1.27 1.27)) hide)
     )
-    (property "Datasheet" "https://www.hirose.com/product/document?clcode=CL0536-0109-0-76&productname=DF13-10P-1.25DSA(76)&series=DF13&documenttype=Catalog&lang=en&documentid=D31687_en" (at 123.19 119.38 0)
+    (property "Datasheet" "" (at 123.19 119.38 0)
       (effects (font (size 1.27 1.27)) hide)
     )
@@
       (effects (font (size 1.27 1.27)) hide)
     )
-    (property "Manufacturer" "Hirose Electric Co Ltd" (at 123.19 119.38 0)
+    (property "Manufacturer" "Samtec" (at 123.19 119.38 0)
       (effects (font (size 1.27 1.27)) hide)
     )
-    (property "Manufacturer Part Number" "DF13-10P-1.25DSA" (at 123.19 119.38 0)
+    (property "Manufacturer Part Number" "T1M-05-GF-DV-K" (at 123.19 119.38 0)
       (effects (font (size 1.27 1.27)) hide)
     )
@@
       (effects (font (size 1.27 1.27)) hide)
     )
-    (property "Supplier Part Number" "H2198-ND" (at 123.19 119.38 0)
+    (property "Supplier Part Number" "SAM15304DKR-ND" (at 123.19 119.38 0)
       (effects (font (size 1.27 1.27)) hide)
     )
